File: PCBs/Control_board/controlBoard_rev0401.sch (KiCad schematic (older format))
At the start: 23 parts, among them J1 Conn_02x03_Odd_Even, U1 ATmega328P-AU, U5 Pi_Header, U6 OLED_I2C, U8 FTDI_Basic, Y1 Crystal

Commit message: Update for BES publication
Parts:
- U8: symbol arduinoBased:FTDI_Basic -> controlBoard_rev0401-rescue:FTDI_Basic-arduinoBased
Other:
- note added: "Revised March 2020 for Publication"
- note removed: "May 15, 2019"
Changed lines of the file:
@@
 IPAX Control Board
 Text Notes 8750 7650 0    60   ~ 12
-May 15, 2019
+Revised March 2020 for Publication
 $Sheet
 S 7250 4500 1650 1000
@@
 	2700 3800 2700 3950
 $Comp
-L arduinoBased:FTDI_Basic U8
+L controlBoard_rev0401-rescue:FTDI_Basic-arduinoBased U8
 U 1 1 5C7DE2F4
 P 6700 6350
