File: PCBs/Control_board/i2c_sensors.sch (KiCad schematic (older format))
At the start: 16 parts, among them J6 Conn_01x04_Male, J7 Conn_01x04_Male, U10 BME280, U7 coin_cell, U9 DS3231MZ

Commit message: Update for revision05a
Parts:
- C10, C12, C14, C16: LCSC (none) -> C15849
- C11, C13, C15, C7: LCSC (none) -> C57112
- J6, J7: footprint Connector_JST:JST_PH_B4B-PH-K_1x04_P2.00mm_Vertical -> conn:conn_1x04_1.5mm
- R28, R29, R30: LCSC (none) -> C25804
- U7: symbol controlBoard_rev0401-rescue:coin_cell-powerReg -> controlBoard_rev05a-rescue:coin_cell-powerReg-controlBoard_rev0401-rescue
Changed lines of the file:
@@
 EESchema Schematic File Version 4
-LIBS:controlBoard_rev0401-cache
+LIBS:controlBoard_rev05a-cache
 EELAYER 26 0
 EELAYER END
 $Descr A4 11693 8268
 encoding utf-8
-Sheet 4 5
+Sheet 5 5
 Title ""
 Date ""
@@
 F 2 "Resistor_SMD:R_0603_1608Metric" V 6090 2240 50  0001 C CNN
 F 3 "~" H 6050 2250 50  0001 C CNN
+F 4 "C25804" H 0   0   50  0001 C CNN "LCSC"
 	1    6050 2250
 	1    0    0    -1
@@
 F 2 "Resistor_SMD:R_0603_1608Metric" V 6390 2240 50  0001 C CNN
 F 3 "~" H 6350 2250 50  0001 C CNN
+F 4 "C25804" H 0   0   50  0001 C CNN "LCSC"
 	1    6350 2250
 	1    0    0    -1
@@
 F 2 "Resistor_SMD:R_0603_1608Metric" V 9690 2090 50  0001 C CNN
 F 3 "~" H 9650 2100 50  0001 C CNN
+F 4 "C25804" H 0   0   50  0001 C CNN "LCSC"
 	1    9650 2100
 	1    0    0    -1
@@
 F 2 "Capacitor_SMD:C_0603_1608Metric" H 7188 1900 50  0001 C CNN
 F 3 "~" H 7150 2050 50  0001 C CNN
+F 4 "C15849" H 0   0   50  0001 C CNN "LCSC"
 	1    7150 2050
 	1    0    0    -1
@@
 F 2 "Capacitor_SMD:C_0603_1608Metric" H 6888 1900 50  0001 C CNN
 F 3 "~" H 6850 2050 50  0001 C CNN
+F 4 "C57112" H 0   0   50  0001 C CNN "LCSC"
 	1    6850 2050
 	1    0    0    -1
@@
 F 2 "Capacitor_SMD:C_0603_1608Metric" H 10538 1900 50  0001 C CNN
 F 3 "~" H 10500 2050 50  0001 C CNN
+F 4 "C15849" H 0   0   50  0001 C CNN "LCSC"
 	1    10500 2050
 	1    0    0    -1
@@
 F 2 "Capacitor_SMD:C_0603_1608Metric" H 10238 1900 50  0001 C CNN
 F 3 "~" H 10200 2050 50  0001 C CNN
+F 4 "C57112" H 0   0   50  0001 C CNN "LCSC"
 	1    10200 2050
 	1    0    0    -1
@@
 F 2 "Capacitor_SMD:C_0603_1608Metric" H 6188 4500 50  0001 C CNN
 F 3 "~" H 6150 4650 50  0001 C CNN
+F 4 "C15849" H 0   0   50  0001 C CNN "LCSC"
 	1    6150 4650
 	1    0    0    -1
@@
 F 2 "Capacitor_SMD:C_0603_1608Metric" H 5888 4500 50  0001 C CNN
 F 3 "~" H 5850 4650 50  0001 C CNN
+F 4 "C57112" H 0   0   50  0001 C CNN "LCSC"
 	1    5850 4650
 	1    0    0    -1
@@
 F 0 "J6" H 4956 4728 50  0000 C CNN
 F 1 "Conn_01x04_Male" H 4956 4637 50  0000 C CNN
-F 2 "Connector_JST:JST_PH_B4B-PH-K_1x04_P2.00mm_Vertical" H 4850 4450 50  0001 C CNN
+F 2 "conn:conn_1x04_1.5mm" H 4850 4450 50  0001 C CNN
 F 3 "~" H 4850 4450 50  0001 C CNN
 	1    4850 4450
@@
 F 2 "Capacitor_SMD:C_0603_1608Metric" H 8538 4500 50  0001 C CNN
 F 3 "~" H 8500 4650 50  0001 C CNN
+F 4 "C15849" H 0   0   50  0001 C CNN "LCSC"
 	1    8500 4650
 	1    0    0    -1
@@
 F 2 "Capacitor_SMD:C_0603_1608Metric" H 8238 4500 50  0001 C CNN
 F 3 "~" H 8200 4650 50  0001 C CNN
+F 4 "C57112" H 0   0   50  0001 C CNN "LCSC"
 	1    8200 4650
 	1    0    0    -1
@@
 F 0 "J7" H 7306 4728 50  0000 C CNN
 F 1 "Conn_01x04_Male" H 7306 4637 50  0000 C CNN
-F 2 "Connector_JST:JST_PH_B4B-PH-K_1x04_P2.00mm_Vertical" H 7200 4450 50  0001 C CNN
+F 2 "conn:conn_1x04_1.5mm" H 7200 4450 50  0001 C CNN
 F 3 "~" H 7200 4450 50  0001 C CNN
 	1    7200 4450
@@
 	7400 4800 8200 4800
 $Comp
-L controlBoard_rev0401-rescue:coin_cell-powerReg U7
+L controlBoard_rev05a-rescue:coin_cell-powerReg-controlBoard_rev0401-rescue U7
 U 1 1 5C54CFE2
 P 3450 2150
