File: PCBs/Control_board/powerControl.sch (KiCad schematic (older format))
At the start: 11 parts, among them J2 Conn_01x02_Male, J3 Conn_01x06_Male, J4 Conn_01x06_Male, U3 NCP361, U4 INA181

Commit message: Update for revision05a
Parts:
- removed C5: 10uF, Capacitor_SMD:C_0805_2012Metric, symbol Device:C
- removed C8: 1000uF, Connector_PinHeader_2.54mm:PinHeader_1x02_P2.54mm_Vertical, symbol Device:C
- removed D3: RED, LED_SMD:LED_0603_1608Metric, symbol Device:LED
- removed R13: 10k, Resistor_SMD:R_0603_1608Metric, symbol Device:R
- removed R3: R, Resistor_SMD:R_1206_3216Metric, symbol Device:R
- removed U3: NCP361, Package_TO_SOT_SMD:SOT-23-5, symbol controlBoard_rev0401-rescue:NCP361-powerReg
- added C5: CP, Connector_PinHeader_2.54mm:PinHeader_1x02_P2.54mm_Vertical, symbol Device:CP
- U4: symbol controlBoard_rev0401-rescue:INA181-powerReg -> controlBoard_rev05a-rescue:INA181-powerReg-controlBoard_rev0401-rescue
Connections:
- net labels added: LED_EN2
- net labels removed: 5V_NPTC, LED_SENSE
- wire segments 50 -> 30
Other:
- moved on the sheet: J2
Changed lines of the file:
@@
 EESchema Schematic File Version 4
-LIBS:controlBoard_rev0401-cache
+LIBS:controlBoard_rev05a-cache
 EELAYER 26 0
 EELAYER END
@@
 Text GLabel 2350 5350 0    60   Input ~ 0
 PI_CTL
-Text Notes 2550 4350 0    60   ~ 0
+Text Notes 2600 4500 0    60   ~ 0
 Pi Power Control
 Wire Wire Line
@@
 L Connector:Conn_01x02_Male J?
 U 1 1 5C0D950E
-P 900 5650
+P 3950 4800
 AR Path="/5C0D950E" Ref="J?"  Part="1"
 AR Path="/5988C2E9/5C0D950E" Ref="J2"  Part="1"
-F 0 "J2" H 1006 5828 50  0000 C CNN
-F 1 "Conn_01x02_Male" H 1006 5737 50  0000 C CNN
-F 2 "Connector_PinHeader_2.54mm:PinHeader_1x02_P2.54mm_Vertical" H 900 5650 50  0001 C CNN
-F 3 "~" H 900 5650 50  0001 C CNN
-	1    900  5650
+F 0 "J2" H 4056 4978 50  0000 C CNN
+F 1 "Conn_01x02_Male" H 4056 4887 50  0000 C CNN
+F 2 "Connector_PinHeader_2.54mm:PinHeader_1x02_P2.54mm_Vertical" H 3950 4800 50  0001 C CNN
+F 3 "~" H 3950 4800 50  0001 C CNN
+	1    3950 4800
 	1    0    0    -1
 $EndComp
@@
 Text Notes 3150 1500 0    59   ~ 0
 Input from power board
-Text GLabel 5550 6250 2    60   Input ~ 0
+Text GLabel 4300 4800 2    60   Input ~ 0
 Vpi
-Text GLabel 1250 5650 2    60   Input ~ 0
-Vpi
-Text GLabel 1250 5750 2    60   Input ~ 0
-5V
-Wire Wire Line
-	1100 5650 1250 5650
-Wire Wire Line
-	1250 5750 1100 5750
-$Comp
-L controlBoard_rev0401-rescue:NCP361-powerReg U3
-U 1 1 5C49578D
-P 4600 6500
-F 0 "U3" H 4750 7015 50  0000 C CNN
-F 1 "NCP361" H 4750 6924 50  0000 C CNN
-F 2 "Package_TO_SOT_SMD:SOT-23-5" H 4750 6600 50  0001 C CNN
-F 3 "DOCUMENTATION" H 4750 6600 50  0001 C CNN
-	1    4600 6500
-	1    0    0    -1
-$EndComp
-Wire Wire Line
-	5550 6250 5400 6250
-Wire Wire Line
-	3600 6250 3750 6250
-$Comp
-L power:GND #PWR?
-U 1 1 5C4986BC
-P 4600 7200
-AR Path="/5BC9CFF4/5C4986BC" Ref="#PWR?"  Part="1"
-AR Path="/5988C2E9/5C4986BC" Ref="#PWR0111"  Part="1"
-F 0 "#PWR0111" H 4600 6950 50  0001 C CNN
-F 1 "GND" H 4600 7050 50  0000 C CNN
-F 2 "" H 4600 7200 50  0000 C CNN
-F 3 "" H 4600 7200 50  0000 C CNN
-	1    4600 7200
-	1    0    0    -1
-$EndComp
-Wire Wire Line
-	4600 7100 4600 7150
-Wire Wire Line
-	4150 6500 4150 7150
-Wire Wire Line
-	4150 7150 4600 7150
-Connection ~ 4600 7150
-Wire Wire Line
-	4600 7150 4600 7200
-$Comp
-L Device:LED D3
-U 1 1 5C49BA33
-P 5700 6500
-F 0 "D3" H 5691 6716 50  0000 C CNN
-F 1 "RED" H 5691 6625 50  0000 C CNN
-F 2 "LED_SMD:LED_0603_1608Metric" H 5700 6500 50  0001 C CNN
-F 3 "~" H 5700 6500 50  0001 C CNN
-	1    5700 6500
-	1    0    0    -1
-$EndComp
-$Comp
-L Device:R R?
-U 1 1 5C49BA96
-P 6150 6500
-AR Path="/5BC9CFF4/5C49BA96" Ref="R?"  Part="1"
-AR Path="/5988C2E9/5C49BA96" Ref="R13"  Part="1"
-F 0 "R13" V 6230 6500 50  0000 C CNN
-F 1 "10k" V 6150 6500 50  0000 C CNN
-F 2 "Resistor_SMD:R_0603_1608Metric" V 6080 6500 50  0001 C CNN
-F 3 "" H 6150 6500 50  0000 C CNN
-	1    6150 6500
-	0    1    1    0
-$EndComp
-Text Label 3650 6250 0    59   ~ 0
-5V_NPTC
-Wire Wire Line
-	5550 6500 5350 6500
-Wire Wire Line
-	5850 6500 6000 6500
-Wire Wire Line
-	6300 6500 6450 6500
-Text Label 6450 6500 0    59   ~ 0
-5V_NPTC
+Text GLabel 4300 4900 2    60   Input ~ 0
+5V
+Wire Wire Line
+	4150 4800 4300 4800
+Wire Wire Line
+	4300 4900 4150 4900
 $Comp
 L Device:R R?
@@
 Wire Wire Line
 	3050 1800 2700 1800
-$Comp
-L Device:C C?
-U 1 1 5C4CFA59
-P 3750 6550
-AR Path="/5BC9CFF4/5C4CFA59" Ref="C?"  Part="1"
-AR Path="/5988C2E9/5C4CFA59" Ref="C5"  Part="1"
-F 0 "C5" H 3865 6596 50  0000 L CNN
-F 1 "10uF" H 3865 6505 50  0000 L CNN
-F 2 "Capacitor_SMD:C_0805_2012Metric" H 3788 6400 50  0001 C CNN
-F 3 "~" H 3750 6550 50  0001 C CNN
-	1    3750 6550
-	1    0    0    -1
-$EndComp
-Text GLabel 5450 6750 2    60   Input ~ 0
+Text GLabel 3800 5250 2    60   Input ~ 0
 Vpi
-Wire Wire Line
-	3750 6250 3750 6400
-Connection ~ 3750 6250
-Wire Wire Line
-	3750 6250 4050 6250
-Wire Wire Line
-	3750 6700 3750 7150
-Wire Wire Line
-	3750 7150 4150 7150
-Connection ~ 4150 7150
 $Comp
 L Connector:Conn_01x06_Male J4
@@
 	5600 1750 5250 1750
 $Comp
-L controlBoard_rev0401-rescue:INA181-powerReg U4
+L controlBoard_rev05a-rescue:INA181-powerReg-controlBoard_rev0401-rescue U4
 U 1 1 5C52284F
 P 7200 3900
@@
 	8100 3750 7800 3750
 Text GLabel 6000 2150 2    59   Input ~ 0
-LED_SENSE
+LED_EN2
 Wire Wire Line
 	6000 2150 5250 2150
-$Comp
-L Device:C C?
-U 1 1 5C4C763B
-P 5150 7000
-AR Path="/5BC9CFF4/5C4C763B" Ref="C?"  Part="1"
-AR Path="/5988C2E9/5C4C763B" Ref="C8"  Part="1"
-F 0 "C8" H 5265 7046 50  0000 L CNN
-F 1 "1000uF" H 5265 6955 50  0000 L CNN
-F 2 "Connector_PinHeader_2.54mm:PinHeader_1x02_P2.54mm_Vertical" H 5188 6850 50  0001 C CNN
-F 3 "~" H 5150 7000 50  0001 C CNN
-	1    5150 7000
-	1    0    0    -1
-$EndComp
-Wire Wire Line
-	5150 7150 4600 7150
-Wire Wire Line
-	5150 6850 5150 6750
-Wire Wire Line
-	5150 6750 5450 6750
 $Sheet
 S 2500 4900 1050 650
@@
 	2300 5000 2500 5000
 Wire Wire Line
-	3550 5250 3600 5250
-Wire Wire Line
-	3600 5250 3600 6250
-$Comp
-L Device:R R3
-U 1 1 5CDC10FE
-P 4700 5600
-F 0 "R3" V 4493 5600 50  0000 C CNN
-F 1 "R" V 4584 5600 50  0000 C CNN
-F 2 "Resistor_SMD:R_1206_3216Metric" V 4630 5600 50  0001 C CNN
-F 3 "~" H 4700 5600 50  0001 C CNN
-	1    4700 5600
-	0    1    1    0
-$EndComp
-Wire Wire Line
-	4550 5600 4050 5600
-Wire Wire Line
-	4050 5600 4050 6250
-Connection ~ 4050 6250
-Wire Wire Line
-	4050 6250 4150 6250
-Wire Wire Line
-	4850 5600 5400 5600
-Wire Wire Line
-	5400 5600 5400 6250
-Connection ~ 5400 6250
-Wire Wire Line
-	5400 6250 5350 6250
+	3550 5250 3800 5250
+$Comp
+L Device:CP C5
+U 1 1 5E8C4AD5
+P 5300 4900
+F 0 "C5" H 5418 4946 50  0000 L CNN
+F 1 "CP" H 5418 4855 50  0000 L CNN
+F 2 "Connector_PinHeader_2.54mm:PinHeader_1x02_P2.54mm_Vertical" H 5338 4750 50  0001 C CNN
+F 3 "~" H 5300 4900 50  0001 C CNN
+	1    5300 4900
+	1    0    0    -1
+$EndComp
+Text GLabel 5400 4700 2    60   Input ~ 0
+Vpi
+$Comp
+L power:GND #PWR?
+U 1 1 5E8C4B17
+P 5300 5150
+AR Path="/5BC9CFF4/5E8C4B17" Ref="#PWR?"  Part="1"
+AR Path="/5988C2E9/5E8C4B17" Ref="#PWR0113"  Part="1"
+F 0 "#PWR0113" H 5300 4900 50  0001 C CNN
+F 1 "GND" H 5300 5000 50  0000 C CNN
+F 2 "" H 5300 5150 50  0000 C CNN
+F 3 "" H 5300 5150 50  0000 C CNN
+	1    5300 5150
+	1    0    0    -1
+$EndComp
+Wire Wire Line
+	5300 4750 5300 4700
+Wire Wire Line
+	5300 4700 5400 4700
+Wire Wire Line
+	5300 5050 5300 5150
 $EndSCHEMATC
