File: PCBs/Control_board/powerFET.sch (KiCad schematic (older format))
At the start: 4 parts, among them Q1 PMOS, Q2 Q_NMOS_GSD

Commit message: Update for revision05a
Parts:
- Q2: LCSC (none) -> C382335
- R4: LCSC (none) -> C23193
- R6: LCSC (none) -> C25804
Changed lines of the file:
@@
 EESchema Schematic File Version 4
-LIBS:controlBoard_rev0401-cache
+LIBS:controlBoard_rev05a-cache
 EELAYER 26 0
 EELAYER END
@@
 F 2 "Resistor_SMD:R_0603_1608Metric" V 4180 4100 50  0001 C CNN
 F 3 "" H 4250 4100 50  0000 C CNN
+F 4 "C23193" H 0   0   50  0001 C CNN "LCSC"
 	1    4250 4100
 	0    1    1    0
@@
 F 2 "Resistor_SMD:R_0603_1608Metric" V 4780 3250 50  0001 C CNN
 F 3 "" H 4850 3250 50  0000 C CNN
+F 4 "C25804" H 0   0   50  0001 C CNN "LCSC"
 	1    4850 3250
 	0    1    1    0
@@
 F 2 "Package_TO_SOT_SMD:SOT-23" H 5100 4200 50  0001 C CNN
 F 3 "~" H 4900 4100 50  0001 C CNN
+F 4 "C382335" H 0   0   50  0001 C CNN "LCSC"
 	1    4900 4100
 	1    0    0    -1
