File: PCBs/Ring_illuminator/ring_illuminator.kicad_pcb (KiCad board)
At the start: 2 copper layers, 60 x 60 mm, 28 parts, among them J1 Conn_01x02_Female, J10 Conn_01x01_Female, J11 Conn_01x01_Female, J12 Conn_01x01_Female, J2 Conn_01x02_Female, J3 Conn_01x01_Female, J4 Conn_01x01_Female, J5 Conn_01x01_Female, J6 Conn_01x01_Female, J7 Conn_01x01_Female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

Commit message: Update for BES publication
Parts:
- removed C1, C2: 22uF, Capacitor_SMD:C_0805_2012Metric
- removed C3, C4: 0.1uF, Capacitor_SMD:C_0603_1608Metric
- removed C5, C6: CP, Capacitor_THT:CP_Radial_D5.0mm_P2.00mm
- removed J2: Conn_01x02_Female, Connector_Molex:Molex_Nano-Fit_105309-xx02_1x02_P2.50mm_Vertical
- added J13: Conn_01x01_Male, conn:large_smd_pad, F.Cu at (-23.0, -12.0)
- added J15: Conn_01x01_Male, conn:large_smd_pad, F.Cu at (23.0, -12.0)
- added J17: Conn_01x01_Male, conn:large_smd_pad, F.Cu at (23.0, 12.0)
- J1: value Conn_01x02_Female -> Conn_01x01_Male; footprint Connector_Molex:Molex_Nano-Fit_105309-xx02_1x02_P2.50mm_Vertical -> conn:large_smd_pad; moved to F.Cu
- moved J1 14.4 mm to (-23.0, 12.0), turned to 0 degrees
Connections:
- D10 pad 1: Net-(D10-Pad1) -> PGND
- D2 pad 2: Net-(D10-Pad1) -> Net-(D1-Pad1)
- D3 pad 2: Net-(D1-Pad1) -> Net-(D2-Pad1)
- D4 pad 1: PGND -> Net-(D4-Pad1)
- D4 pad 2: Net-(D2-Pad1) -> Net-(D3-Pad1)
- D5 pad 1: Net-(D5-Pad1) -> PGND
- D5 pad 2: Net-(D3-Pad1) -> Net-(D4-Pad1)
- D7 pad 2: Net-(D5-Pad1) -> Net-(D6-Pad1)
- D8 pad 1: Net-(D10-Pad2) -> Net-(D8-Pad1)
- D8 pad 2: Net-(D6-Pad1) -> Net-(D7-Pad1)
- D9 pad 1: PGND -> Net-(D10-Pad2)
- D9 pad 2: Net-(D7-Pad1) -> Net-(D8-Pad1)
- J1 pad 1: VLED2 -> PGND
Routing:
- net PGND: track 129.5 -> 14.9 mm
- net Net-(D5-Pad1): track 36.9 -> 0.00 mm, vias 5 -> 0
- net Net-(D10-Pad1): track 26.2 -> 0.00 mm
- net Net-(D3-Pad1): track 43.0 -> 20.4 mm
- net Net-(D4-Pad1): track 0.00 -> 19.5 mm
- net Net-(D7-Pad1): track 28.9 -> 13.0 mm
- net Net-(D10-Pad2): track 26.2 -> 13.1 mm
- net Net-(D6-Pad1): track 25.9 -> 13.0 mm
- net Net-(D2-Pad1): track 32.6 -> 22.2 mm
- net Net-(D8-Pad1): track 0.00 -> 10.3 mm
- net VLED1: track 22.4 -> 13.6 mm, vias 1 -> 0
- net Net-(D1-Pad1): track 35.5 -> 28.8 mm
- net VLED2: track 19.7 -> 15.0 mm, vias 1 -> 0
- removed copper zone on B.Cu, net PGND
Other:
- board text added: "Rev02a"
- board text added: "V+"
- board text added: "V-"
- board text removed: "Rev03a"

Commit message: Update for revision05a
Parts:
- removed J15, J17: Conn_01x01_Male, conn:large_smd_pad
- added J14: Conn_01x01_Female, conn:large_smd_pad, F.Cu at (-8.00, 26.0)
- added J2: Conn_01x01_Female, conn:large_smd_pad, F.Cu at (8.00, -26.0)
- J1, J13: value Conn_01x01_Male -> Conn_01x01_Female
- moved J1 51.4 mm to (27.0, 0.00), turned to 180 degrees
- moved J13 12.6 mm to (-27.0, 0.00), turned to 180 degrees
Connections:
- net VLED2 renamed LED2+
- D1 pad 2: VLED1 -> LED1+
- D10 pad 1: PGND -> Net-(D10-Pad1)
- D2 pad 2: Net-(D1-Pad1) -> Net-(D10-Pad1)
- D3 pad 2: Net-(D2-Pad1) -> Net-(D1-Pad1)
- D4 pad 1: Net-(D4-Pad1) -> LED2-
- D4 pad 2: Net-(D3-Pad1) -> Net-(D2-Pad1)
- D5 pad 1: PGND -> Net-(D5-Pad1)
- D5 pad 2: Net-(D4-Pad1) -> Net-(D3-Pad1)
- D7 pad 2: Net-(D6-Pad1) -> Net-(D5-Pad1)
- D8 pad 1: Net-(D8-Pad1) -> Net-(D10-Pad2)
- D8 pad 2: Net-(D7-Pad1) -> Net-(D6-Pad1)
- D9 pad 1: Net-(D10-Pad2) -> LED1-
- D9 pad 2: Net-(D8-Pad1) -> Net-(D7-Pad1)
- J1 pad 1: PGND -> LED1+
Routing:
- net Net-(D5-Pad1): track 0.00 -> 41.5 mm
- net Net-(D10-Pad1): track 0.00 -> 26.2 mm
- net Net-(D3-Pad1): track 20.4 -> 42.0 mm
- net Net-(D4-Pad1): track 19.5 -> 0.00 mm
- net Net-(D7-Pad1): track 13.0 -> 28.1 mm
- net PGND: track 14.9 -> 0.00 mm
- net VLED1: track 13.6 -> 0.00 mm
- net Net-(D6-Pad1): track 13.0 -> 25.9 mm
- net Net-(D10-Pad2): track 13.1 -> 24.1 mm
- net LED2+: track 15.0 -> 4.35 mm
- net Net-(D2-Pad1): track 22.2 -> 32.6 mm
- net LED1+: track 0.00 -> 10.4 mm
- net Net-(D8-Pad1): track 10.3 -> 0.00 mm
- net LED2-: track 0.00 -> 7.23 mm
- net LED1-: track 0.00 -> 5.81 mm
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- removed copper zone on F.Cu, net PGND
Other:
- board text added: "Rev03b"
- board text added: "V1+"
- board text added: "V1-"
- board text added: "V2+"
- board text added: "V2-"
- board text removed: "Rev02a"
- board text removed: "V+"
- board text removed: "V-"
